File: kicad_magicsub1590b.kicad_pcb (KiCad board)
At the start: 2 copper layers, 56 x 56 mm, 18 parts, among them P1 EXT_IO, P2 EXT_IO, P3 M3Drill, P4 M3Drill, P5 EXT_IO, P6 M3Drill, P7 M3Drill, P8 EXT_IO, U1 B10k, U2 B10k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

Commit message: 配線引いた
Parts:
- added G***: LOGO, hastech:LogiClover, B.Cu at (147.0, 86.6)
- moved C2 0.60 mm to (140.6, 75.5), turned to 180 degrees
Routing:
- net GND: track 23.5 -> 298.8 mm, vias 0 -> 41
- net /ADC_Vref: track 0.00 -> 82.1 mm, vias 0 -> 3
- net /MIDI_TX_5: track 0.00 -> 67.3 mm, vias 0 -> 1
- net /MIDI_RX_5: track 0.00 -> 62.9 mm
- net /MIDI_TX_4: track 0.00 -> 62.6 mm
- net +5V: track 0.00 -> 58.4 mm
- net /MIDI_RX_4: track 0.00 -> 58.3 mm
- net /EN_5V: track 0.00 -> 58.2 mm
- net +12V: track 0.00 -> 54.9 mm
- net /ADC_2: track 11.6 -> 59.3 mm
- net /ADC_1: track 0.00 -> 46.4 mm
- net /GPI_0: track 0.00 -> 38.1 mm
- net /GPI_2: track 0.00 -> 33.3 mm
- net /GPI_1: track 0.00 -> 33.1 mm
- net /GPI_3: track 0.00 -> 27.5 mm
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- added copper zone on B.Cu, net GND
- added copper zone on F.Cu, net GND
Other:
- board text added: "12V"
- board text added: "ADC:0"
- board text added: "ADC:1"
- board text added: "ADC:2"
- board text added: "EN:5V"
- board text added: "GND"
- board text added: "I:0"
- board text added: "I:1"
- board text added: "I:2"
- board text added: "I:3"
- board text added: "IN_L"
- board text added: "IN_R"
- board text added: "L"
- board text added: "MIC"
- board text added: "MIDI RX"
- board text added: "MIDI TX"
- board text added: "Magic UserInterface"
- board text added: "O:3"
- board text added: "O:4"
- board text added: "O:5"
- board text added: "OUT[2:0]"
- board text added: "OUT_L"
- board text added: "OUT_R"
- board text added: "R"
- board text added: "Rev.A"
